File: Cad setup/test.kicad_sch (KiCad schematic)
At the start: 8 parts, among them SW1 SW_Push, SW2 SW_Push, SW3 SW_Push

Commit message: updated cad file to allign with new setup
Connections:
- net at A1.17 (D2): now also R1.1
- net at A1.18 (D3): no longer R1.1
- net at A1.19 (D4): now also R2.1
- net at A1.20 (D5): no longer R2.1
- net at A1.21 (D6): no longer R3.1
- net at A1.22 (D7): now also R3.1
Changed lines of the file:
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@@
-	(wire
-		(pts
-			(xy 114.3 71.12) (xy 129.54 71.12)
-		)
-		(stroke
-			(width 0)
-			(type default)
-		)
-	)
 	(wire
 		(pts
@@
 	(wire
 		(pts
-			(xy 106.68 68.58) (xy 106.68 77.47)
+			(xy 106.68 66.04) (xy 106.68 77.47)
 		)
 		(stroke
@@
 	(wire
 		(pts
-			(xy 129.54 63.5) (xy 99.06 63.5)
-		)
-		(stroke
-			(width 0)
-			(type default)
-		)
-	)
-	(wire
-		(pts
 			(xy 68.58 49.53) (xy 68.58 59.69)
 		)
@@
 	(wire
 		(pts
-			(xy 99.06 63.5) (xy 99.06 73.66)
+			(xy 99.06 60.96) (xy 99.06 73.66)
 		)
 		(stroke
@@
 	(wire
 		(pts
-			(xy 106.68 68.58) (xy 129.54 68.58)
+			(xy 129.54 66.04) (xy 106.68 66.04)
+		)
+		(stroke
+			(width 0)
+			(type default)
+		)
+	)
+	(wire
+		(pts
+			(xy 129.54 73.66) (xy 114.3 73.66)
 		)
 		(stroke
@@
 	(wire
 		(pts
-			(xy 114.3 71.12) (xy 114.3 81.28)
-		)
-		(stroke
-			(width 0)
-			(type default)
-		)
-	)
-	(wire
-		(pts
 			(xy 129.54 81.28) (xy 124.46 81.28)
 		)
@@
 	(wire
 		(pts
+			(xy 114.3 73.66) (xy 114.3 81.28)
+		)
+		(stroke
+			(width 0)
+			(type default)
+		)
+	)
+	(wire
+		(pts
 			(xy 68.58 59.69) (xy 68.58 109.22)
 		)
@@
 		)
 		(stroke
+			(width 0)
+			(type default)
+		)
+	)
+	(wire
+		(pts
+			(xy 129.54 60.96) (xy 99.06 60.96)
+		)
+		(stroke
